File: kicad/pille.kicad_sch (KiCad schematic)
At the start: 0 parts

Commit message: a
Signed-off-by: Zbigniew Opiol <opiol.zbigniew@gmail.com>
Other:
- added sheet MCU (mcu.kicad_sch)
Changed lines of the file:
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@@
+    )
+  )
+  (sheet (at 112.141 80.137) (size 29.718 28.194) (fields_autoplaced)
+    (stroke (width 0.1524) (type solid))
+    (fill (color 0 0 0 0.0000))
+    (property "Sheetname" "MCU" (at 112.141 79.4254 0)
+      (effects (font (size 1.27 1.27)) (justify left bottom))
+    )
+    (property "Sheetfile" "mcu.kicad_sch" (at 112.141 108.9156 0)
+      (effects (font (size 1.27 1.27)) (justify left top))
+    )
+    (instances
+      (project "pille"
+        (path "/d0b7719a-58de-4781-915d-11143b3f1d8a" (page "3"))
+      )
     )
   )
